File: 2017-2018/lec-buzzer_alt.sch (EAGLE design)
At the start: 27 parts, among them U1 74HC595PW, U2 74HC595PW, U3 DRV2605LDGSR, U4 ATMEGA328P-AUR, U5 74HC595PW, U6 74HC595PW, X1 2X3SHROUDED, X2 MINI-USB-32005-201

Commit message: Testcode
Other:
- note added: "I2C Pulls"
- note added: "Make Button into interrupt"
Changed lines of the file:
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@@
 <?xml version="1.0" encoding="utf-8"?>
 <!DOCTYPE eagle SYSTEM "eagle.dtd">
-<eagle version="8.3.2">
+<eagle version="8.4.0">
 <drawing>
 <settings>
@@
 <setting verticaltext="up"/>
 </settings>
-<grid distance="0.05" unitdist="inch" unit="inch" style="lines" multiple="1" display="no" altdistance="0.01" altunitdist="inch" altunit="inch"/>
+<grid distance="0.1" unitdist="inch" unit="inch" style="lines" multiple="1" display="no" altdistance="0.01" altunitdist="inch" altunit="inch"/>
 <layers>
 <layer number="1" name="Top" color="4" fill="1" visible="no" active="no"/>
@@
 <wire x1="327.66" y1="147.32" x2="414.02" y2="147.32" width="0.1524" layer="103" style="shortdash"/>
 <text x="330.2" y="139.7" size="3.81" layer="103" font="vector">Indicator LED</text>
+<text x="38.1" y="124.46" size="1.778" layer="98">I2C Pulls</text>
+<text x="83.82" y="81.28" size="1.778" layer="91">Make Button into interrupt</text>
 </plain>
 <instances>
